Commit message: added launch file to visualize the URDF file with rviz2

File: mm_ws/src/mobile_manipulator_description/urdf/mobile_manipulator.urdf.xacro (robot description, xacro)
@@ -3,3 +3,49 @@
     <xacro:include filename="$(find mobile_manipulator_description)/urdf/properties.xacro" />
     <xacro:include filename="$(find mobile_manipulator_description)/urdf/inertia.xacro" />
+    <!-- LINKS -->
+    <link name="base_footprint" />
+    <link name="base_link">
+        <visual>
+            <origin xyz="0 0 ${chassis_height/2}" rpy="0 0 0" />
+            <geometry>
+                <box size="${chassis_length} ${chassis_width} ${chassis_height}" />
+            </geometry>
+            <material name="blue_acrylic" />
+        </visual>
+        <collision>
+            <origin xyz="0 0 ${chassis_height/2}" rpy="0 0 0" />
+            <geometry>
+                <box size="${chassis_length} ${chassis_width} ${chassis_height}" />
+            </geometry>
+        </collision>
+        <xacro:box_inertia m="${chassis_mass}" x="${chassis_length}" y="${chassis_width}" z="${chassis_height}" />
+    </link>
+    <link name="base_left_wheel_link">
+        <visual>
+            <origin xyz="0 0 0" rpy="${pi/2} 0 0" />
+            <geometry>
+                <cylinder radius="${wheel_radius}" length="${wheel_width}" />
+            </geometry>
+            <material name="black_rubber" />
+        </visual>
+        <collision>
+            <origin xyz="0 0 0" rpy="0 0 0" />
+            <geometry>
+                <cylinder radius="${wheel_radius}" length="${wheel_width}" />
+            </geometry>
+        </collision>
+        <xacro:cylinder_inertia m="${wheel_mass}" r="${wheel_radius}" h="${wheel_width}" />
+    </link>
+    <!-- JOINTS -->
+    <joint name="base_to_footprint" type="fixed">
+        <parent link="base_footprint"/>
+        <child link="base_link"/>
+        <origin xyz="0 0 ${wheel_radius}" rpy="0 0 0"/>
+    </joint>
+    <joint name="base_to_left_wheel_joint" type="continuous">
+        <parent link="base_link"/>
+        <child link="base_left_wheel_link"/>
+        <origin xyz="${chassis_length/4 - 0.01} ${chassis_width/2+wheel_width/2} 0" rpy="0 0 0"/>
+        <axis xyz="0 1 0"/>
+    </joint>
 </robot>

Commit message: URDF for differential drive mobile robot

File: mm_ws/src/mobile_manipulator_description/urdf/mobile_manipulator.urdf.xacro (robot description, xacro)
@@ -21,5 +21,5 @@
         <xacro:box_inertia m="${chassis_mass}" x="${chassis_length}" y="${chassis_width}" z="${chassis_height}" />
     </link>
-    <link name="base_left_wheel_link">
+    <link name="left_wheel_link">
         <visual>
             <origin xyz="0 0 0" rpy="${pi/2} 0 0" />
@@ -30,10 +30,42 @@
         </visual>
         <collision>
-            <origin xyz="0 0 0" rpy="0 0 0" />
+            <origin xyz="0 0 0" rpy="${pi/2} 0 0" />
             <geometry>
                 <cylinder radius="${wheel_radius}" length="${wheel_width}" />
             </geometry>
         </collision>
-        <xacro:cylinder_inertia m="${wheel_mass}" r="${wheel_radius}" h="${wheel_width}" />
+        <xacro:wheel_inertia m="${wheel_mass}" r="${wheel_radius}" h="${wheel_width}" />
+    </link>
+    <link name="right_wheel_link">
+        <visual>
+            <origin xyz="0 0 0" rpy="${pi/2} 0 0" />
+            <geometry>
+                <cylinder radius="${wheel_radius}" length="${wheel_width}" />
+            </geometry>
+            <material name="black_rubber" />
+        </visual>
+        <collision>
+            <origin xyz="0 0 0" rpy="${pi/2} 0 0" />
+            <geometry>
+                <cylinder radius="${wheel_radius}" length="${wheel_width}" />
+            </geometry>
+        </collision>
+        <xacro:wheel_inertia m="${wheel_mass}" r="${wheel_radius}" h="${wheel_width}" />
+    </link>
+    <link name="caster_wheel_link">
+        <visual>
+            <origin xyz="0 0 0" rpy="0 0 0" />
+            <geometry>
+                <sphere radius="${caster_radius}" />
+            </geometry>
+            <material name="grey_caster" />
+        </visual>
+        <collision>
+            <origin xyz="0 0 0" rpy="0 0 0" />
+            <geometry>
+                <sphere radius="${caster_radius}" />
+            </geometry>
+        </collision>
+        <xacro:sphere_inertia m="${caster_mass}" r="${caster_radius}" />
     </link>
     <!-- JOINTS -->
@@ -45,7 +77,18 @@
     <joint name="base_to_left_wheel_joint" type="continuous">
         <parent link="base_link"/>
-        <child link="base_left_wheel_link"/>
-        <origin xyz="${chassis_length/4 - 0.01} ${chassis_width/2+wheel_width/2} 0" rpy="0 0 0"/>
+        <child link="left_wheel_link"/>
+        <origin xyz="${-chassis_length/4 + 0.01} ${chassis_width/2+wheel_width/2} 0" rpy="0 0 0"/>
         <axis xyz="0 1 0"/>
     </joint>
+    <joint name="base_to_right_wheel_joint" type="continuous">
+        <parent link="base_link"/>
+        <child link="right_wheel_link"/>
+        <origin xyz="${-chassis_length/4 + 0.01} ${-chassis_width/2-wheel_width/2} 0" rpy="0 0 0"/>
+        <axis xyz="0 1 0"/>
+    </joint>
+    <joint name="base_to_caster_wheel_joint" type="fixed">
+        <parent link="base_link"/>
+        <child link="caster_wheel_link"/>
+        <origin xyz="${chassis_length/4} 0 ${-caster_radius}" rpy="0 0 0"/>
+    </joint>
 </robot>

Commit message: Added Robotic Arm Description - URDF

File: mm_ws/src/mobile_manipulator_description/urdf/mobile_manipulator.urdf.xacro (robot description, xacro)
@@ -19,5 +19,8 @@
             </geometry>
         </collision>
-        <xacro:box_inertia m="${chassis_mass}" x="${chassis_length}" y="${chassis_width}" z="${chassis_height}" />
+        <xacro:box_inertia m="${chassis_mass}"
+                            x="${chassis_length}"
+                            y="${chassis_width}"
+                            z="${chassis_height}" />
     </link>
     <link name="left_wheel_link">
@@ -59,5 +62,5 @@
                 <sphere radius="${caster_radius}" />
             </geometry>
-            <material name="grey_caster" />
+            <material name="grey" />
         </visual>
         <collision>
@@ -92,4 +95,6 @@
         <origin xyz="${chassis_length/4} 0 ${-caster_radius}" rpy="0 0 0"/>
     </joint>
+    <!-- Robotic Arm -->
+    <xacro:include filename="$(find mobile_manipulator_description)/urdf/robotic_arm.xacro" />
     <!-- GAZEBO SETUP: Plugin Configuration -->
     <xacro:include filename="$(find mobile_manipulator_description)/urdf/gazebo_setup.xacro" />

File: mm_ws/src/mobile_manipulator_description/urdf/properties.xacro (robot description, xacro)
@@ -12,4 +12,9 @@
     <!-- Caster wheel -->
     <xacro:property name="caster_radius"    value="0.025"/>
+    <!-- Robotic Arm -->
+    <xacro:property name="arm_base_length" value="0.05"/>
+    <xacro:property name="arm_base_height" value="0.01"/>
+    <xacro:property name="arm_link_length" value="0.15"/>
+    <xacro:property name="arm_link_radius" value="0.01"/>
     <!-- Mass values (kg) -->
     <xacro:property name="chassis_mass"     value="3"/>

Commit message: Changes in some materials tag

File: mm_ws/src/mobile_manipulator_description/urdf/mobile_manipulator.urdf.xacro (robot description, xacro)
@@ -62,5 +62,5 @@
                 <sphere radius="${caster_radius}" />
             </geometry>
-            <material name="grey" />
+            <material name="grey_caster" />
         </visual>
         <collision>

File: mm_ws/src/mobile_manipulator_description/urdf/properties.xacro (robot description, xacro)
@@ -31,3 +31,9 @@
         <color rgba="0.6 0.6 0.6 1.0"/>
     </material>
+    <material name="orange">
+        <color rgba="1.0 0.5 0.0 1.0"/>
+    </material>
+    <material name="yellow">
+        <color rgba="1.0 1.0 0.0 1.0"/>
+    </material>
 </robot>
